File: STM32_XTW2_CLONE.kicad_sch (KiCad schematic)
At the start: 26 parts, among them J1 USB A MALE, J2 ST-LINK, SW1 RST, U1 STM32F103C8Tx, U2 AMS1117-3.3, Y1 8Mhz

Commit message: 25/03/23/C
Parts:
- added D3: LED, LED_SMD:LED_1206_3216Metric, symbol Device:LED
- added R7: 1K, Resistor_SMD:R_1206_3216Metric, symbol Device:R
Connections:
- net GND: now also D3.1 (K)
- net at R4.2: now also U1.38 (PA15); no longer U1.43 (PB7)
- new net: D3.2 (A), R7.1
- new net: R7.2, U1.43 (PB7)
- no-connect marks 24 -> 23
Other:
- moved on the sheet: D2, R4
Changed lines of the file:
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@@
     (title "Clone XTW-2")
     (date "2023-03-08")
-    (rev "1.2V")
+    (rev "1.2.1V")
     (company "xDNA Electronics & Design")
   )
@@
   (no_connect (at 68.58 121.92))
   (no_connect (at 68.58 93.98))
-  (no_connect (at 101.6 93.98))
   (no_connect (at 68.58 106.68))
   (no_connect (at 68.58 96.52))
@@
     (stroke (width 0) (type default))
   )
+  (wire (pts (xy 101.6 93.98) (xy 104.14 93.98))
+    (stroke (width 0) (type default))
+  )
   (wire (pts (xy 49.53 101.6) (xy 55.88 101.6))
     (stroke (width 0) (type default))
@@
     (stroke (width 0) (type dash_dot_dot))
   )
+  (wire (pts (xy 129.54 101.6) (xy 128.27 101.6))
+    (stroke (width 0) (type default))
+  )
   (wire (pts (xy 83.82 50.8) (xy 83.82 48.26))
     (stroke (width 0) (type default))
@@
     (stroke (width 0) (type dash_dot_dot))
   )
+  (wire (pts (xy 120.65 101.6) (xy 114.3 101.6))
+    (stroke (width 0) (type default))
+  )
   (wire (pts (xy 137.16 165.1) (xy 137.16 167.64))
     (stroke (width 0) (type default))
@@
     (stroke (width 0) (type default))
   )
+  (wire (pts (xy 104.14 93.98) (xy 104.14 101.6))
+    (stroke (width 0) (type default))
+  )
   (wire (pts (xy 78.74 165.1) (xy 78.74 167.64))
     (stroke (width 0) (type default))
   )
   (wire (pts (xy 57.15 88.9) (xy 68.58 88.9))
+    (stroke (width 0) (type default))
+  )
+  (wire (pts (xy 106.68 101.6) (xy 104.14 101.6))
     (stroke (width 0) (type default))
   )
@@
     )
   )
+  (symbol (lib_id "Device:LED") (at 45.72 101.6 0) (unit 1)
+    (in_bom yes) (on_board yes) (dnp no) (fields_autoplaced)
+    (property "Reference" "D3" (at 44.1325 96.52 0)
+      (effects (font (size 1.27 1.27)))
+    )
+    (property "Value" "LED" (at 44.1325 99.06 0)
+      (effects (font (size 1.27 1.27)))
+    )
+    (property "Footprint" "LED_SMD:LED_1206_3216Metric" (at 45.72 101.6 0)
+      (effects (font (size 1.27 1.27)) hide)
+    )
+    (property "Datasheet" "~" (at 45.72 101.6 0)
+      (effects (font (size 1.27 1.27)) hide)
+    )
+    (pin "1")
+    (pin "2")
+    (instances
+      (project "STM32_XTW2_CLONE"
+        (path "/e342adb5-bb9c-4c9d-bdeb-4fcac8de750c"
+          (reference "D3") (unit 1)
+        )
+      )
+    )
+  )
   (symbol (lib_id "Device:R") (at 53.975 54.61 90) (unit 1)
     (in_bom yes) (on_board yes) (dnp no)
@@
     )
   )
-  (symbol (lib_id "Device:R") (at 59.69 101.6 90) (unit 1)
+  (symbol (lib_id "Device:R") (at 110.49 101.6 270) (unit 1)
     (in_bom yes) (on_board yes) (dnp no)
-    (property "Reference" "R4" (at 59.69 101.6 90)
-      (effects (font (size 1.27 1.27)))
-    )
-    (property "Value" "1K" (at 59.69 99.06 90)
-      (effects (font (size 1.27 1.27)))
-    )
-    (property "Footprint" "Resistor_SMD:R_1206_3216Metric" (at 59.69 103.378 90)
-      (effects (font (size 1.27 1.27)) hide)
-    )
-    (property "Datasheet" "~" (at 59.69 101.6 0)
+    (property "Reference" "R4" (at 110.49 101.6 90)
+      (effects (font (size 1.27 1.27)))
+    )
+    (property "Value" "1K" (at 110.49 104.14 90)
+      (effects (font (size 1.27 1.27)))
+    )
+    (property "Footprint" "Resistor_SMD:R_1206_3216Metric" (at 110.49 99.822 90)
+      (effects (font (size 1.27 1.27)) hide)
+    )
+    (property "Datasheet" "~" (at 110.49 101.6 0)
       (effects (font (size 1.27 1.27)) hide)
     )
@@
     )
   )
+  (symbol (lib_id "Device:R") (at 59.69 101.6 90) (unit 1)
+    (in_bom yes) (on_board yes) (dnp no)
+    (property "Reference" "R7" (at 59.69 101.6 90)
+      (effects (font (size 1.27 1.27)))
+    )
+    (property "Value" "1K" (at 59.69 99.06 90)
+      (effects (font (size 1.27 1.27)))
+    )
+    (property "Footprint" "Resistor_SMD:R_1206_3216Metric" (at 59.69 103.378 90)
+      (effects (font (size 1.27 1.27)) hide)
+    )
+    (property "Datasheet" "~" (at 59.69 101.6 0)
+      (effects (font (size 1.27 1.27)) hide)
+    )
+    (pin "1")
+    (pin "2")
+    (instances
+      (project "STM32_XTW2_CLONE"
+        (path "/e342adb5-bb9c-4c9d-bdeb-4fcac8de750c"
+          (reference "R7") (unit 1)
+        )
+      )
+    )
+  )
   (symbol (lib_id "power:GND") (at 127 190.5 0) (unit 1)
     (in_bom yes) (on_board yes) (dnp no) (fields_autoplaced)
@@
         (path "/e342adb5-bb9c-4c9d-bdeb-4fcac8de750c"
           (reference "#PWR06") (unit 1)
+        )
+      )
+    )
+  )
+  (symbol (lib_id "power:GND") (at 129.54 101.6 90) (unit 1)
+    (in_bom yes) (on_board yes) (dnp no) (fields_autoplaced)
+    (property "Reference" "#PWR028" (at 135.89 101.6 0)
+      (effects (font (size 1.27 1.27)) hide)
+    )
+    (property "Value" "GND" (at 133.35 101.6 0)
+      (effects (font (size 1.27 1.27)))
+    )
+    (property "Footprint" "" (at 129.54 101.6 0)
+      (effects (font (size 1.27 1.27)) hide)
+    )
+    (property "Datasheet" "" (at 129.54 101.6 0)
+      (effects (font (size 1.27 1.27)) hide)
+    )
+    (pin "1")
+    (instances
+      (project "STM32_XTW2_CLONE"
+        (path "/e342adb5-bb9c-4c9d-bdeb-4fcac8de750c"
+          (reference "#PWR028") (unit 1)
         )
       )
@@
     )
   )
-  (symbol (lib_id "Device:LED") (at 45.72 101.6 0) (unit 1)
-    (in_bom yes) (on_board yes) (dnp no) (fields_autoplaced)
-    (property "Reference" "D2" (at 44.1325 96.52 0)
-      (effects (font (size 1.27 1.27)))
-    )
-    (property "Value" "LED" (at 44.1325 99.06 0)
-      (effects (font (size 1.27 1.27)))
-    )
-    (property "Footprint" "LED_SMD:LED_1206_3216Metric" (at 45.72 101.6 0)
-      (effects (font (size 1.27 1.27)) hide)
-    )
-    (property "Datasheet" "~" (at 45.72 101.6 0)
-      (effects (font (size 1.27 1.27)) hide)
-    )
+  (symbol (lib_id "Device:LED") (at 124.46 101.6 180) (unit 1)
+    (in_bom yes) (on_board yes) (dnp no) (fields_autoplaced)
+    (property "Reference" "D2" (at 126.0475 106.68 0)
+      (effects (font (size 1.27 1.27)))
+    )
+    (property "Value" "LED" (at 126.0475 104.14 0)
+      (effects (font (size 1.27 1.27)))
+    )
+    (property "Footprint" "LED_SMD:LED_1206_3216Metric" (at 124.46 101.6 0)
+      (effects (font (size 1.27 1.27)) hide)
+    )
+    (property "Datasheet" "~" (at 124.46 101.6 0)
+      (effects (font (size 1.27 1.27)) hide)
+    )
